File: pcb/hotwire-lite.sch (KiCad schematic (older format))
At the start: 24 parts, among them J1 Barrel_Jack, J2 Conn_01x02, J4 Conn_01x04, J5 Screw_Terminal_01x02, Q1 Si4162DY, SW1 SW_Push, U1 AP1117-50, U2 INA181

Commit message: updated pcb
Parts:
- added R3: 10k, Resistor_SMD:R_0805_2012Metric, symbol Device:R_Small_US
- added R6: 220, Resistor_SMD:R_0805_2012Metric, symbol Device:R_Small_US
- C3: value 1uF -> 0.1uF
- TP1: renamed from volt1; value TestPoint -> volt
- TP2: renamed from vin1; value TestPoint -> vin
- TP3: renamed from reg1; value TestPoint -> reg
- TP4: renamed from pwm1; value TestPoin -> pwm
- TP5: renamed from amp1; value TestPoint -> amp
- renumbered J5 to J2, J4 to J3, J2 to J4, R5 to R4, R3 to R5, R4 to R7, MCU1 to U2, U2 to U3
Connections:
- net GNDREF: now also J3.1 (Pin_1), R3.2; no longer J3.4 (Pin_4), R2.2
- net UPDI: now also J3.4 (Pin_4); no longer J3.1 (Pin_1)
- net pwm_output: now also R6.1; no longer Q1.4 (G), TP4.1
- net rx_button: now also J3.3 (Pin_3); no longer J3.2 (Pin_2)
- net tx_led: now also J3.2 (Pin_2); no longer J3.3 (Pin_3)
- net vin: no longer R1.1
- net voltage_sense: now also R2.2, R3.1; no longer R1.2, R2.1
- net shunt_low: now reaches J4.1 (Pin_1), R7.2, U3.4 (-)
- net shunt_low: now also R1.1
- new net: Q1.4 (G), R6.2, TP4.1
- new net: R1.2, R2.1
Other:
- moved on the sheet: C4, J3, J4, Q1, R7, TP1, TP4, TP5, U3
