File: pcb/hotwire-lite.kicad_sch (KiCad schematic)
At the start: 23 parts, among them J1 wire_pos, J2 wire_neg, J3 Barrel_Jack, Q1 SIRA18ADP, SW1 SW_Push, U1 NCP716B, U2 ATtiny402-SS, U3 INA181A1

Commit message: v1.0 hardware
Parts:
- removed H1: MountingHole_Pad, MountingHole:MountingHole_3.2mm_M3_Pad_Via, symbol Mechanical:MountingHole_Pad
- removed J1: wire_pos, hotwire-lite:Wire Solder Pad, symbol Connector_Generic:Conn_01x01
- removed J3: Barrel_Jack, Connector_BarrelJack:BarrelJack_CLIFF_FC681465S_SMT_Horizontal, symbol Connector:Barrel_Jack
- removed Q1: SIRA18ADP, Package_SO:Vishay_PowerPAK_1212-8_Single, symbol hotwire-lite:SIRA18ADP
- removed R1, R2, R3, R4: 1k, Resistor_SMD:R_0603_1608Metric, symbol Device:R_US
- removed R6: 0.050, Resistor_SMD:R_2512_6332Metric, symbol Device:R_US
- removed TP6: DBG, TestPoint:TestPoint_Pad_D1.0mm, symbol Connector:TestPoint
- removed TP7: rx, TestPoint:TestPoint_Pad_D1.0mm, symbol Connector:TestPoint
- removed TP8: tx, TestPoint:TestPoint_Pad_D1.0mm, symbol Connector:TestPoint
- removed U1: NCP716B, Package_TO_SOT_SMD:SOT-23-5, symbol hotwire-lite:NCP716B
- added J1: (no value), symbol Connector:Barrel_Jack_Switch_Pin3Ring
- added J3: (no value), symbol Connector_Generic:Conn_01x01
- added Q1: (no value), symbol hotwire-lite:SiRA18ADP
- added R1, R2, R3, R4, R6: (no value), symbol Device:R_Small_US
- added TP1, TP2, TP3: (no value), symbol Connector:TestPoint
- added U1: (no value), symbol hotwire-lite:NCP716
- C1, C2: value 1uF -> (none); footprint Capacitor_SMD:C_0603_1608Metric -> (none)
- C3: value 0.01uF -> (none); footprint Capacitor_SMD:C_0603_1608Metric -> (none)
- C4: value 0.1uF -> (none); footprint Capacitor_SMD:C_0603_1608Metric -> (none)
- D1: value LED -> (none); footprint LED_SMD:LED_0805_2012Metric -> (none)
- J2: value wire_neg -> (none); footprint hotwire-lite:Wire Solder Pad -> (none)
- R5: value 1k -> (none); footprint Resistor_SMD:R_0603_1608Metric -> (none)
- SW1: value SW_Push -> (none); footprint Button_Switch_SMD:SW_SPST_PTS645 -> (none)
- U2: value ATtiny402-SS -> (none)
- U3: value INA181A1 -> (none); footprint Package_TO_SOT_SMD:SOT-23-6 -> (none)
Connections:
- net shunt_low is gone; now on net wire_pos: U3.4 (-)
- net +5V: now also C3.2, C4.2, U1.3 (VOUT); no longer C3.1, C4.1
- net GND: now also C3.1, C4.1, J1.2, J1.3, Q1.1 (S), Q1.2 (S), Q1.3 (S), R3.2, R4.2, U1.1 (GND); no longer C3.2, C4.2
- net UPDI: now also TP1.1
- net rx_button: now also TP2.1
- net tx_led: now also TP3.1
- net vin: now also J1.1, R6.1, U1.2 (VIN)
- net voltage_sense: now also R2.2, R3.1
- net at R5.2: now also Q1.4 (G)
- net at D1.1 (K): now also R4.1
- net load_neg renamed wire_pos
- net wire_pos: now also R1.1, R6.2
- new net: R1.2, R2.1
- new net wire_neg: J3.1 (Pin_1), Q1.5 (D)
Other:
- note added: "current amplifier"
- note added: "indicator LED"
- note added: "pad connections"
- note added: "power input"
- note added: "voltage divider"
- note removed: "TODO: replace with correct FET"
- note removed: "UART test points"
- note removed: "hotwire connection"
- note removed: "switching and current sense"
- note removed: "transmit LED"
- note removed: "voltage input and regulation"
- note removed: "voltage sense divider"
- title: Hotwire Controller Lite -> (none)
